File: Hardware/STM32F4/STM32F4_Breakout.kicad_sch (KiCad schematic)
At the start: 50 parts, among them J1 Screw_Terminal_01x02, J2 SWD, J3 Conn_01x04, J4 Conn_01x04, J5 USB_B, Q1 AO3401A, SW1 SW_SPDT, U1 STM32F405RGT6, U2 MP2303ADN, U3 USBLC6-2SC6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

Commit message: Consolidated Kicad projects
Connections:
- net GND: no longer C11.1, R2.2, Y1.3
- new net: C11.1, R2.2, Y1.3
- no-connect marks 40 -> 5
Changed lines of the file:
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@@
-	)
-	(junction
-		(at 114.3 146.05)
-		(diameter 0)
-		(color 0 0 0 0)
 	)
 	(junction
@@
 	)
 	(no_connect
-		(at 40.64 144.78)
-	)
-	(no_connect
-		(at 40.64 139.7)
-	)
-	(no_connect
-		(at 40.64 111.76)
-	)
-	(no_connect
-		(at 40.64 119.38)
-	)
-	(no_connect
-		(at 76.2 116.84)
-	)
-	(no_connect
-		(at 40.64 142.24)
-	)
-	(no_connect
-		(at 40.64 127)
-	)
-	(no_connect
-		(at 76.2 149.86)
-	)
-	(no_connect
-		(at 40.64 124.46)
-	)
-	(no_connect
-		(at 40.64 147.32)
-	)
-	(no_connect
-		(at 76.2 139.7)
-	)
-	(no_connect
-		(at 40.64 134.62)
-	)
-	(no_connect
-		(at 76.2 111.76)
-	)
-	(no_connect
-		(at 76.2 93.98)
-	)
-	(no_connect
-		(at 76.2 119.38)
-	)
-	(no_connect
-		(at 76.2 101.6)
-	)
-	(no_connect
-		(at 40.64 152.4)
-	)
-	(no_connect
-		(at 76.2 96.52)
-	)
-	(no_connect
-		(at 76.2 172.72)
-	)
-	(no_connect
-		(at 76.2 104.14)
-	)
-	(no_connect
-		(at 76.2 109.22)
-	)
-	(no_connect
-		(at 76.2 132.08)
-	)
-	(no_connect
-		(at 76.2 137.16)
-	)
-	(no_connect
-		(at 76.2 142.24)
-	)
-	(no_connect
 		(at 198.12 72.39)
 	)
@@
 	)
 	(no_connect
-		(at 40.64 116.84)
-	)
-	(no_connect
 		(at 109.22 31.75)
-	)
-	(no_connect
-		(at 76.2 106.68)
-	)
-	(no_connect
-		(at 76.2 147.32)
-	)
-	(no_connect
-		(at 40.64 154.94)
-	)
-	(no_connect
-		(at 40.64 149.86)
-	)
-	(no_connect
-		(at 40.64 132.08)
 	)
 	(no_connect
@@
 	)
 	(no_connect
-		(at 40.64 137.16)
-	)
-	(no_connect
-		(at 76.2 175.26)
-	)
-	(no_connect
-		(at 40.64 129.54)
-	)
-	(no_connect
 		(at 109.22 36.83)
 	)
-	(no_connect
-		(at 76.2 114.3)
-	)
-	(no_connect
-		(at 40.64 121.92)
-	)
 	(wire
 		(pts
@@
 	(wire
 		(pts
-			(xy 114.3 143.51) (xy 114.3 146.05)
-		)
-		(stroke
-			(width 0)
-			(type default)
-		)
-	)
-	(wire
-		(pts
 			(xy 58.42 185.42) (xy 58.42 187.96)
 		)
@@
 	(wire
 		(pts
-			(xy 114.3 146.05) (xy 114.3 152.4)
-		)
-		(stroke
+			(xy 114.3 143.51) (xy 114.3 152.4)
+		)
+		(stroke

Commit message: CAN transceiver
Parts:
- added J8: CAN Connector1, Connector_Molex:Molex_Mega-Fit_76829-0006_2x03_P5.70mm_Vertical, symbol Connector_Generic:Conn_02x03_Top_Bottom
- added J9: CAN Connector2, Connector_Molex:Molex_Mega-Fit_76829-0006_2x03_P5.70mm_Vertical, symbol Connector_Generic:Conn_02x03_Top_Bottom
- added R12, R13: 120, Resistor_SMD:R_0603_1608Metric_Pad0.98x0.95mm_HandSolder, symbol Device:R_Small
- added U4, U5: TJA1051T, Package_SO:SOIC-8_3.9x4.9mm_P1.27mm, symbol Interface_CAN_LIN:TJA1051T
Connections:
- net +5V: now also J8.4 (Pin_4), J9.4 (Pin_4), U4.3 (VCC), U5.3 (VCC)
- net CAN1_RX: now also U4.4 (RXD)
- net CAN1_TX: now also U4.1 (TXD)
- net CAN2_RX: now also U5.4 (RXD)
- net CAN2_TX: now also U5.1 (TXD)
- net GND: now also J8.6 (Pin_6), J9.6 (Pin_6), U4.2 (GND), U5.2 (GND)
- net CAN SIlent Mode 1: now reaches U1.35 (PB14)
- net CAN SIlent Mode 1: now also U4.8 (S)
- net CAN SIlent Mode 2: now reaches U1.36 (PB15)
- net CAN SIlent Mode 2: now also U5.8 (S)
- new net CAN1+: J8.1 (Pin_1), R12.2, U4.7 (CANH)
- new net CAN1-: J8.2 (Pin_2), R12.1, U4.6 (CANL)
- new net CAN2+: J9.1 (Pin_1), R13.2, U5.7 (CANH)
- new net CAN2-: J9.2 (Pin_2), R13.1, U5.6 (CANL)
- no-connect marks 5 -> 42
